Commit message: fix

File: cartesian_description/urdf/cartesian_cell.xacro (robot description, xacro)
@@ -5,6 +5,6 @@
   <joint name="world2cartesian" type="fixed">
     <parent link="world"/>
-    <child link="link_Z"/>
-    <origin xyz="0 0 0.5"/>
+    <child link="link_X"/>
+    <origin xyz="0.5 0 0.0"/>
   </joint>
 </robot>

File: cartesian_description/urdf/cartesian_robot.urdf.xacro (robot description, xacro)
@@ -2,93 +2,63 @@
 <robot xmlns:xacro="http://ros.org/wiki/xacro" name="cartesian_robot" >
   <material name="blue">
-    <color rgba="0 0 0.8 1"/>
+    <color rgba="0 0 1 0.5"/>
+  </material>
+  <material name="green">
+    <color rgba="0 1 0 0.5"/>
+  </material>
+  <material name="red">
+    <color rgba="1 0 0 0.5"/>
   </material>
   <material name="black">
     <color rgba="0 0 0 1"/>
   </material>
-  <material name="white">
-    <color rgba="1 1 1 1"/>
-  </material>
-  <link name="link_Z">
-    <visual>
-      <geometry>
-        <cylinder length="1" radius="0.05"/>
-      </geometry>
-      <origin rpy="0 0 0" xyz="0 0 0"/>
-      <material name="blue"/>
-    </visual>
-    <collision>
-      <origin rpy="0 0 0" xyz="0 0 0"/>
-      <geometry>
-        <sphere radius="0.0"/>
-      </geometry>
-    </collision>
-  </link>
-  <link name="link_Y">
-    <visual>
-      <geometry>
-        <cylinder length="1" radius="0.05"/>
-      </geometry>
-      <origin rpy="1.570795 0 0" xyz="0 0 0"/>
-      <material name="black"/>
-    </visual>
-    <collision>
-      <origin rpy="1.570795 0 0" xyz="0 0 0"/>
-      <geometry>
-        <sphere radius="0.0"/>
-      </geometry>
-    </collision>
-  </link>
-  <joint name="from_Z_to_Y" type="prismatic">
-    <parent link="link_Z"/>
-    <child link="link_Y"/>
-    <axis xyz = "0 0 1" />
-    <origin rpy="0 0 0" xyz="0 0.5 -0.5"/>
-    <limit effort="1000.0" lower="0" upper="1" velocity="0.5"/>
-  </joint>
-  <link name="link_fake">
-    <visual>
-      <geometry>
-        <sphere radius="0.00005"/>
-      </geometry>
-      <origin rpy="0 0 0" xyz="0 0 0"/>
-      <material name="black"/>
-    </visual>
-    <collision>
-      <origin rpy="0.0 0.0 0.0" xyz="0 0 0"/>
-      <geometry>
-        <sphere radius="0.0"/>
-      </geometry>
-    </collision>
-  </link>
-  <joint name="from_Y_to_fake" type="prismatic">
-    <parent link="link_Y"/>
-    <child link="link_fake"/>
-    <axis xyz = "0 1 0" />
-    <origin rpy="0 0 0" xyz="0 -0.5 0"/>
-    <limit effort="1000.0" lower="0" upper="1" velocity="0.5"/>
-  </joint>
-  <link name="link_X">
-    <visual>
-      <geometry>
-        <cylinder length="1" radius="0.05"/>
-      </geometry>
-      <origin rpy="0 -1.570795 0" xyz="0 0 0"/>
-      <material name="white"/>
-    </visual>
-    <collision>
-      <origin rpy="0 -1.570795 0" xyz="0 0 0"/>
-      <geometry>
-        <sphere radius="0.0"/>
-      </geometry>
-    </collision>
-  </link>
-  <joint name="from_fake_to_X" type="prismatic">
-    <parent link="link_fake"/>
-    <child link="link_X"/>
-    <axis xyz = "1 0 0" />
-    <origin rpy="0 0 0" xyz="-0.5 0 0"/>
-    <limit effort="1000.0" lower="0" upper="1" velocity="0.5"/>
-  </joint>
+  <link name="link_Z"/>
+  <link name="link_Y"/>
+  <link name="link_X"/>
+  <!-- <link name="link_Z">
+  <visual>
+    <geometry>
+      <cylinder length="1" radius="0.05"/>
+    </geometry>
+    <origin rpy="0 0 0" xyz="0 0 0"/>
+    <material name="blue"/>
+  </visual>
+  <collision>
+    <origin rpy="0 0 0" xyz="0 0 0"/>
+    <geometry>
+      <sphere radius="0.0"/>
+    </geometry>
+  </collision>
+</link> -->
+<!-- <link name="link_Y">
+  <visual>
+    <geometry>
+      <cylinder length="1" radius="0.05"/>
+    </geometry>
+    <origin rpy="1.570795 0 0" xyz="0 0 0"/>
+    <material name="green"/>
+  </visual>
+  <collision>
+    <origin rpy="1.570795 0 0" xyz="0 0 0"/>
+    <geometry>
+      <sphere radius="0.0"/>
+    </geometry>
+  </collision>
+</link> -->
+<!-- <link name="link_X">
+  <visual>
+    <geometry>
+      <cylinder length="1" radius="0.05"/>
+    </geometry>
+    <origin rpy="0 -1.570795 0" xyz="0 0 0"/>
+    <material name="red"/>
+  </visual>
+  <collision>
+    <origin rpy="0 -1.570795 0" xyz="0 0 0"/>
+    <geometry>
+      <sphere radius="0.0"/>
+    </geometry>
+  </collision>
+</link> -->
   <link name="end_effector">
     <visual>
@@ -106,8 +76,24 @@
     </collision>
   </link>
-  <joint name="from_X_to_end" type="fixed">
+  <joint name="joint_X" type="prismatic">
     <parent link="link_X"/>
+    <child link="link_Y"/>
+    <axis xyz = "1 0 0" />
+    <origin rpy="0 0 0" xyz="-0.5 0.5 0"/>
+    <limit effort="1000.0" lower="0" upper="1" velocity="0.5"/>
+  </joint>
+  <joint name="joint_Y" type="prismatic">
+    <parent link="link_Y"/>
+    <child link="link_Z"/>
+    <axis xyz = "0 1 0" />
+    <origin rpy="0 0 0" xyz="0 -0.5 0.5"/>
+    <limit effort="1000.0" lower="0" upper="1" velocity="0.5"/>
+  </joint>
+  <joint name="joint_Z" type="prismatic">
+    <parent link="link_Z"/>
     <child link="end_effector"/>
-    <origin rpy="0 0 0" xyz="0.5 0 0"/>
+    <axis xyz = "0 0 1" />
+    <origin rpy="0 0 0" xyz="0 0 -0.5"/>
+    <limit effort="1000.0" lower="0" upper="1" velocity="0.5"/>
   </joint>
 </robot>

Commit message: UAV cell

File: cartesian_description/urdf/cartesian_cell.xacro (robot description, xacro)
@@ -1,10 +1,13 @@
 <?xml version="1.0"?>
 <robot xmlns:xacro="http://ros.org/wiki/xacro" name="cartesian_cell" >
-<xacro:include filename="$(find cartesian_description)/urdf/cartesian_robot.urdf.xacro" />
-  <link name="world"/>
-  <joint name="world2cartesian" type="fixed">
-    <parent link="world"/>
-    <child link="link_X"/>
-    <origin xyz="0.5 0 0.0"/>
-  </joint>
+<xacro:include filename="$(find cartesian_description)/urdf/base_cell.xacro" />
+<xacro:base_cell
+  lb_X   = "0.0"
+  ub_X   = "1.0"
+  lb_Y   = "0.0"
+  ub_Y   = "1.0"
+  lb_Z   = "0.0"
+  ub_Z   = "1.0"
+  radius = "0.005"
+/>
 </robot>

File: cartesian_description/urdf/cartesian_robot.urdf.xacro (robot description, xacro)
@@ -1,4 +1,17 @@
 <?xml version="1.0"?>
 <robot xmlns:xacro="http://ros.org/wiki/xacro" name="cartesian_robot" >
+  <xacro:macro name="cartesian_robot" params="
+     ub_X:=1.0
+     lb_X:=0.0
+     ub_Y:=1.0
+     lb_Y:=0.0
+     ub_Z:=1.0
+     lb_Z:=0.0
+     radius:=0.005">
+  <xacro:property name="velocity" value="0.5" />
+  <xacro:property name="effort" value="1000.0"/>
+  <xacro:property name="mid_point_X" value="${(ub_X-lb_X)/2.0}" />
+  <xacro:property name="mid_point_Y" value="${(ub_Y-lb_Y)/2.0}" />
+  <xacro:property name="mid_point_Z" value="${(ub_Z-lb_Z)/2.0}" />
   <material name="blue">
     <color rgba="0 0 1 0.5"/>
@@ -16,53 +29,8 @@
   <link name="link_Y"/>
   <link name="link_X"/>
-  <!-- <link name="link_Z">
-  <visual>
-    <geometry>
-      <cylinder length="1" radius="0.05"/>
-    </geometry>
-    <origin rpy="0 0 0" xyz="0 0 0"/>
-    <material name="blue"/>
-  </visual>
-  <collision>
-    <origin rpy="0 0 0" xyz="0 0 0"/>
-    <geometry>
-      <sphere radius="0.0"/>
-    </geometry>
-  </collision>
-</link> -->
-<!-- <link name="link_Y">
-  <visual>
-    <geometry>
-      <cylinder length="1" radius="0.05"/>
-    </geometry>
-    <origin rpy="1.570795 0 0" xyz="0 0 0"/>
-    <material name="green"/>
-  </visual>
-  <collision>
-    <origin rpy="1.570795 0 0" xyz="0 0 0"/>
-    <geometry>
-      <sphere radius="0.0"/>
-    </geometry>
-  </collision>
-</link> -->
-<!-- <link name="link_X">
-  <visual>
-    <geometry>
-      <cylinder length="1" radius="0.05"/>
-    </geometry>
-    <origin rpy="0 -1.570795 0" xyz="0 0 0"/>
-    <material name="red"/>
-  </visual>
-  <collision>
-    <origin rpy="0 -1.570795 0" xyz="0 0 0"/>
-    <geometry>
-      <sphere radius="0.0"/>
-    </geometry>
-  </collision>
-</link> -->
   <link name="end_effector">
     <visual>
       <geometry>
-        <sphere radius="0.005"/>
+        <sphere radius="${radius}"/>
       </geometry>
       <origin rpy="0 0 0" xyz="0 0 0"/>
@@ -72,5 +40,5 @@
       <origin rpy="0 0 0" xyz="0 0 0"/>
       <geometry>
-        <sphere radius="0.005"/>
+        <sphere radius="${radius}"/>
       </geometry>
     </collision>
@@ -80,6 +48,6 @@
     <child link="link_Y"/>
     <axis xyz = "1 0 0" />
-    <origin rpy="0 0 0" xyz="-0.5 0.5 0"/>
-    <limit effort="1000.0" lower="0" upper="1" velocity="0.5"/>
+    <origin rpy="0 0 0" xyz="${-mid_point_X} ${mid_point_Y} 0"/>
+    <limit effort="${effort}" lower="${lb_X}" upper="${ub_X}" velocity="${velocity}"/>
   </joint>
   <joint name="joint_Y" type="prismatic">
@@ -87,6 +55,6 @@
     <child link="link_Z"/>
     <axis xyz = "0 1 0" />
-    <origin rpy="0 0 0" xyz="0 -0.5 0.5"/>
-    <limit effort="1000.0" lower="0" upper="1" velocity="0.5"/>
+    <origin rpy="0 0 0" xyz="0 ${-mid_point_Y} ${mid_point_Z}"/>
+    <limit effort="${effort}" lower="${lb_Y}" upper="${ub_Y}" velocity="${velocity}"/>
   </joint>
   <joint name="joint_Z" type="prismatic">
@@ -94,6 +62,7 @@
     <child link="end_effector"/>
     <axis xyz = "0 0 1" />
-    <origin rpy="0 0 0" xyz="0 0 -0.5"/>
-    <limit effort="1000.0" lower="0" upper="1" velocity="0.5"/>
+    <origin rpy="0 0 0" xyz="0 0 ${-mid_point_Z}"/>
+    <limit effort="${effort}" lower="${lb_Z}" upper="${ub_Z}" velocity="${velocity}"/>
   </joint>
+</xacro:macro>
 </robot>
