Commit message: galileo : added maze scenario and faulty controller. debugged gazebo integration. works correctly

File: cartesian_description/urdf/base_cell.xacro (robot description, xacro)
@@ -12,5 +12,5 @@
   <xacro:if value="${dim == 2}">
     <xacro:include filename="$(find cartesian_description)/urdf/planar_robot.urdf.xacro" />
-    <xacro:cartesian_robot
+    <xacro:planar_robot
       lb_X   = "${lb_X}"
       ub_X   = "${ub_X}"

File: cartesian_description/urdf/planar_robot.urdf.xacro (robot description, xacro)
@@ -1,5 +1,5 @@
 <?xml version="1.0"?>
-<robot xmlns:xacro="http://ros.org/wiki/xacro" name="cartesian_robot" >
-  <xacro:macro name="cartesian_robot" params="
+<robot xmlns:xacro="http://ros.org/wiki/xacro" name="planar_robot" >
+  <xacro:macro name="planar_robot" params="
      ub_X:=1.0
      lb_X:=0.0

File: planar_robot/planar_robot_description/urdf/planar_robot.xacro (robot description, xacro)
@@ -20,3 +20,4 @@
     <xacro:add_gazebo_addons/>
   </xacro:if>
+  <xacro:include filename="$(find planar_robot_description)/urdf/scenarios/maze_1.xacro" />
 </robot>
