Commit message: galileo : tested with gazebo (added self collisions) and tested faulty controller

File: cartesian_description/urdf/planar_robot.urdf.xacro (robot description, xacro)
@@ -8,5 +8,5 @@
      radius:=0.005">
   <xacro:property name="velocity" value="0.5" />
-  <xacro:property name="effort" value="1000.0"/>
+  <xacro:property name="effort" value="1.0"/>
   <xacro:property name="mid_point_X" value="${(ub_X-lb_X)/2.0}" />
   <xacro:property name="mid_point_Y" value="${(ub_Y-lb_Y)/2.0}" />
@@ -29,5 +29,5 @@
       <mass value="0.000001"/>
       <inertia
-     ixx="0.00001" ixy="0.0" ixz="0.0" iyy="0.00001" iyz="0.0" izz="0.00001"/>
+     ixx="0.00000001" ixy="0.0" ixz="0.0" iyy="0.00000001" iyz="0.0" izz="0.00000001"/>
     </inertial>
   </link>
@@ -37,5 +37,5 @@
       <mass value="0.000001"/>
       <inertia
-     ixx="0.00001" ixy="0.0" ixz="0.0" iyy="0.00001" iyz="0.0" izz="0.00001"/>
+     ixx="0.00000001" ixy="0.0" ixz="0.0" iyy="0.00000001" iyz="0.0" izz="0.00000001"/>
     </inertial>
   </link>
@@ -62,4 +62,5 @@
     <origin rpy="0 0 0" xyz="${-mid_point_X} ${mid_point_Y} 0"/>
     <limit effort="${effort}" lower="${lb_X}" upper="${ub_X}" velocity="${velocity}"/>
+    <dynamics damping="0.01" friction="0.01"/>
   </joint>
   <joint name="joint_Y" type="prismatic">
@@ -69,4 +70,5 @@
     <origin rpy="0 0 0" xyz="0.0 ${-mid_point_Y} 0.0"/>
     <limit effort="${effort}" lower="${lb_Y}" upper="${ub_Y}" velocity="${velocity}"/>
+    <dynamics damping="0.01" friction="0.01"/>
   </joint>
 </xacro:macro>

File: planar_robot/planar_robot_description/urdf/planar_robot.xacro (robot description, xacro)
@@ -19,4 +19,7 @@
     <xacro:include filename="$(find planar_robot_description)/urdf/gazebo_integration.xacro"/>
     <xacro:add_gazebo_addons/>
+    <gazebo>
+      <self_collide>true</self_collide>
+    </gazebo>
   </xacro:if>
   <xacro:include filename="$(find planar_robot_description)/urdf/scenarios/maze_1.xacro" />

File: planar_robot/planar_robot_description/urdf/scenarios/maze_1.xacro (robot description, xacro)
@@ -33,7 +33,7 @@
       </collision>
       <inertial>
-        <mass value="1.0"/>
+        <mass value="100000.0"/>
         <origin xyz="0 0 ${wall_height / 2}" rpy="0 0 0"/>
-        <inertia ixx="0.1" ixy="0" ixz="0" iyy="0.1" iyz="0" izz="0.1"/>
+        <inertia ixx="1000" ixy="0" ixz="0" iyy="1000" iyz="0" izz="1000"/>
       </inertial>
     </link>
@@ -63,5 +63,5 @@
       </collision>
       <inertial>
-        <mass value="1.0"/>
+        <mass value="100000.0"/>
         <origin xyz="0 0 ${pillar_height / 2}" rpy="0 0 0"/>
         <inertia ixx="0.01" ixy="0" ixz="0" iyy="0.01" iyz="0" izz="0.01"/>
