Commit message: galileo : added different scenarios to planar cartesian robot

File: planar_robot/planar_robot_description/urdf/planar_robot.ros2_control.xacro (robot description, xacro)
@@ -18,5 +18,5 @@
                 <command_interface name="velocity"/>
                 <state_interface name="position">
-                  <param name="initial_value">0.0</param>
+                  <param name="initial_value">0.1</param>
                 </state_interface>
                 <state_interface name="velocity"/>
@@ -26,5 +26,5 @@
                 <command_interface name="velocity"/>
                 <state_interface name="position">
-                  <param name="initial_value">0.0</param>
+                  <param name="initial_value">0.1</param>
                 </state_interface>
                 <state_interface name="velocity"/>

File: planar_robot/planar_robot_description/urdf/planar_robot.xacro (robot description, xacro)
@@ -3,4 +3,6 @@
   <xacro:arg name="use_gazebo" default="false"/>
   <xacro:property name="use_gazebo" value="$(arg use_gazebo)"/>
+  <xacro:arg name="scenario" default="maze_2"/>
+  <xacro:property name="scenario" value="$(arg scenario)"/>
   <xacro:include filename="$(find cartesian_description)/urdf/base_cell.xacro" />
   <xacro:base_cell
@@ -23,4 +25,4 @@
     </gazebo>
   </xacro:if>
-  <xacro:include filename="$(find planar_robot_description)/urdf/scenarios/maze_1.xacro" />
+  <xacro:include filename="$(find planar_robot_description)/urdf/scenarios/${scenario}.xacro" />
 </robot>

File: planar_robot/planar_robot_description/urdf/scenarios/maze_0.xacro (robot description, xacro)
@@ -8,5 +8,4 @@
   <xacro:property name="x_offset" value="0.5"/>
   <xacro:property name="y_offset" value="0.5"/>
-  <xacro:property name="box_height" value="0.1"/>
   <link name="maze_base_link"/>
   <joint name="maze_world_joint" type="fixed">
@@ -75,34 +74,4 @@
     </joint>
   </xacro:macro>
-  <!-- === Parameterized Box Obstacle Macro === -->
-  <xacro:macro name="maze_box" params="name x y size">
-    <link name="${name}_link">
-      <visual>
-        <origin xyz="0 0 ${box_height / 2}" rpy="0 0 0"/>
-        <geometry>
-          <box size="${size} ${size} ${box_height}"/>
-        </geometry>
-        <material name="red">
-          <color rgba="0.8 0.2 0.2 1.0"/>
-        </material>
-      </visual>
-      <collision>
-        <origin xyz="0 0 ${box_height / 2}" rpy="0 0 0"/>
-        <geometry>
-          <box size="${size} ${size} ${box_height}"/>
-        </geometry>
-      </collision>
-      <inertial>
-        <mass value="1000.0"/>
-        <origin xyz="0 0 ${size / 2}" rpy="0 0 0"/>
-        <inertia ixx="1" ixy="0" ixz="0" iyy="1" iyz="0" izz="1"/>
-      </inertial>
-    </link>
-    <joint name="${name}_joint" type="fixed">
-      <parent link="maze_base_link"/>
-      <child link="${name}_link"/>
-      <origin xyz="${x} ${y} 0" rpy="0 0 0"/>
-    </joint>
-  </xacro:macro>
   <!-- === Outer square (1x1m boundary) === -->
   <xacro:maze_wall name="boundary_top"    length="1.0" x="0.0" y="0.5" yaw="0.0"/>
@@ -110,8 +79,17 @@
   <xacro:maze_wall name="boundary_left"   length="1.0" x="-0.5" y="0.0" yaw="1.5708"/>
   <xacro:maze_wall name="boundary_right"  length="1.0" x="0.5" y="0.0" yaw="1.5708"/>
-  <!-- === Dour Box Obstacles === -->
-  <xacro:maze_box name="box_1" x="-0.2" y="0.2" size="0.2"/>
-  <xacro:maze_box name="box_2" x="0.2" y="0.2" size="0.2"/>
-  <xacro:maze_box name="box_3" x="-0.2" y="-0.2" size="0.2"/>
-  <xacro:maze_box name="box_4" x="0.2" y="-0.2" size="0.2"/>
+  <!-- === Ten inner walls === -->
+  <xacro:maze_wall name="wall_1" length="0.3" x="-0.3" y="0.3" yaw="0.0"/>
+  <xacro:maze_wall name="wall_2" length="0.2" x="-0.1" y="0.4" yaw="1.5708"/>
+  <xacro:maze_wall name="wall_3" length="0.4" x="0.2"  y="0.3" yaw="0.0"/>
+  <xacro:maze_wall name="wall_4" length="0.3" x="0.0"  y="0.0" yaw="1.5708"/>
+  <xacro:maze_wall name="wall_5" length="0.2" x="0.2"  y="-0.1" yaw="0.0"/>
+  <xacro:maze_wall name="wall_6" length="0.4" x="-0.3" y="-0.2" yaw="0.0"/>
+  <xacro:maze_wall name="wall_7" length="0.3" x="0.3"  y="-0.3" yaw="1.5708"/>
+  <xacro:maze_wall name="wall_8" length="0.2" x="-0.4" y="0.1" yaw="1.5708"/>
+  <xacro:maze_wall name="wall_9" length="0.2" x="0.4"  y="0.1" yaw="1.5708"/>
+  <xacro:maze_wall name="wall_10" length="0.4" x="0.0" y="-0.4" yaw="0.0"/>
+  <!-- === Pillars === -->
+  <xacro:maze_pillar name="pillar_1" x="-0.25" y="-0.25"/>
+  <xacro:maze_pillar name="pillar_2" x="0.25" y="0.25"/>
 </robot>

File: planar_robot/planar_robot_description/urdf/scenarios/maze_2.xacro (robot description, xacro)
@@ -110,8 +110,12 @@
   <xacro:maze_wall name="boundary_left"   length="1.0" x="-0.5" y="0.0" yaw="1.5708"/>
   <xacro:maze_wall name="boundary_right"  length="1.0" x="0.5" y="0.0" yaw="1.5708"/>
-  <!-- === Dour Box Obstacles === -->
-  <xacro:maze_box name="box_1" x="-0.2" y="0.2" size="0.2"/>
-  <xacro:maze_box name="box_2" x="0.2" y="0.2" size="0.2"/>
-  <xacro:maze_box name="box_3" x="-0.2" y="-0.2" size="0.2"/>
-  <xacro:maze_box name="box_4" x="0.2" y="-0.2" size="0.2"/>
+  <!-- === Eight Box Obstacles === -->
+  <xacro:maze_box name="box_1" x="-0.25" y="-0.25" size="0.15"/>
+  <xacro:maze_box name="box_2" x="-0.25" y="0.0" size="0.15"/>
+  <xacro:maze_box name="box_3" x="-0.25" y="0.25" size="0.15"/>
+  <xacro:maze_box name="box_4" x="0.0" y="-0.25" size="0.15"/>
+  <xacro:maze_box name="box_5" x="0.0" y="0.0" size="0.15"/>
+  <xacro:maze_box name="box_6" x="0.0" y="0.25" size="0.15"/>
+  <xacro:maze_box name="box_7" x="0.25" y="0.0" size="0.15"/>
+  <xacro:maze_box name="box_8" x="0.25" y="0.25" size="0.15"/>
 </robot>
